File: cap64pcb/cap64pcb.kicad_sch (KiCad schematic)
At the start: 29 parts, among them J1 SM05B_SURS_TF, Q1 BSS138, Q2 BSS138, U1 MPR121QR2, U2 SPX3819M5-L-3-3

Commit message: shifted PTH up on touch pads
Parts:
- TP1: footprint cap_pads:CAPPAD_7.6x7.6_Chevron_1 -> cap_pads:CAPPAD_7.6x7.6_Chevron_1_TopPTH
- TP10, TP11, TP2, TP3, TP4, TP5, TP8, TP9: footprint cap_pads:CAPPAD_7.6x7.6_Chevron_2 -> cap_pads:CAPPAD_7.6x7.6_Chevron_2_TopPTH
- TP12: footprint cap_pads:CAPPAD_7.6x7.6_Chevron_3 -> cap_pads:CAPPAD_7.6x7.6_Chevron_3_TopPTH
- TP7: footprint cap_pads:CAPPAD_7.6x7.6_Chevron_2_shifted -> cap_pads:CAPPAD_7.6x7.6_Chevron_2_TopPTH
Changed lines of the file:
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@@
       (effects (font (size 1.27 1.27)) (justify left) hide)
     )
-    (property "Footprint" "cap_pads:CAPPAD_7.6x7.6_Chevron_3" (id 2) (at 127 79.375 0)
+    (property "Footprint" "cap_pads:CAPPAD_7.6x7.6_Chevron_3_TopPTH" (id 2) (at 127 79.375 0)
       (effects (font (size 1.27 1.27)) hide)
     )
@@
       (effects (font (size 1.27 1.27)) (justify left) hide)
     )
-    (property "Footprint" "cap_pads:CAPPAD_7.6x7.6_Chevron_2" (id 2) (at 127 71.755 0)
+    (property "Footprint" "cap_pads:CAPPAD_7.6x7.6_Chevron_2_TopPTH" (id 2) (at 127 71.755 0)
       (effects (font (size 1.27 1.27)) hide)
     )
@@
       (effects (font (size 1.27 1.27)) (justify left) hide)
     )
-    (property "Footprint" "cap_pads:CAPPAD_7.6x7.6_Chevron_2" (id 2) (at 127 69.215 0)
+    (property "Footprint" "cap_pads:CAPPAD_7.6x7.6_Chevron_2_TopPTH" (id 2) (at 127 69.215 0)
       (effects (font (size 1.27 1.27)) hide)
     )
@@
       (effects (font (size 1.27 1.27)) (justify left) hide)
     )
-    (property "Footprint" "cap_pads:CAPPAD_7.6x7.6_Chevron_2" (id 2) (at 127 76.835 0)
+    (property "Footprint" "cap_pads:CAPPAD_7.6x7.6_Chevron_2_TopPTH" (id 2) (at 127 76.835 0)
       (effects (font (size 1.27 1.27)) hide)
     )
@@
       (effects (font (size 1.27 1.27)) (justify left) hide)
     )
-    (property "Footprint" "cap_pads:CAPPAD_7.6x7.6_Chevron_2" (id 2) (at 127 56.515 0)
+    (property "Footprint" "cap_pads:CAPPAD_7.6x7.6_Chevron_2_TopPTH" (id 2) (at 127 56.515 0)
       (effects (font (size 1.27 1.27)) hide)
     )
@@
       (effects (font (size 1.27 1.27)) (justify left) hide)
     )
-    (property "Footprint" "cap_pads:CAPPAD_7.6x7.6_Chevron_2" (id 2) (at 127 61.595 0)
+    (property "Footprint" "cap_pads:CAPPAD_7.6x7.6_Chevron_2_TopPTH" (id 2) (at 127 61.595 0)
       (effects (font (size 1.27 1.27)) hide)
     )
@@
       (effects (font (size 1.27 1.27)) (justify left) hide)
     )
-    (property "Footprint" "cap_pads:CAPPAD_7.6x7.6_Chevron_2" (id 2) (at 127 53.975 0)
+    (property "Footprint" "cap_pads:CAPPAD_7.6x7.6_Chevron_2_TopPTH" (id 2) (at 127 53.975 0)
       (effects (font (size 1.27 1.27)) hide)
     )
@@
       (effects (font (size 1.27 1.27)) (justify left) hide)
     )
-    (property "Footprint" "cap_pads:CAPPAD_7.6x7.6_Chevron_2_shifted" (id 2) (at 127 66.675 0)
+    (property "Footprint" "cap_pads:CAPPAD_7.6x7.6_Chevron_2_TopPTH" (id 2) (at 127 66.675 0)
       (effects (font (size 1.27 1.27)) hide)
     )
@@
       (effects (font (size 1.27 1.27)) (justify left) hide)
     )
-    (property "Footprint" "cap_pads:CAPPAD_7.6x7.6_Chevron_2" (id 2) (at 127 59.055 0)
+    (property "Footprint" "cap_pads:CAPPAD_7.6x7.6_Chevron_2_TopPTH" (id 2) (at 127 59.055 0)
       (effects (font (size 1.27 1.27)) hide)
     )
@@
       (effects (font (size 1.27 1.27)) (justify left) hide)
     )
-    (property "Footprint" "cap_pads:CAPPAD_7.6x7.6_Chevron_1" (id 2) (at 127 51.435 0)
+    (property "Footprint" "cap_pads:CAPPAD_7.6x7.6_Chevron_1_TopPTH" (id 2) (at 127 51.435 0)
       (effects (font (size 1.27 1.27)) hide)
     )
@@
       (effects (font (size 1.27 1.27)) (justify left) hide)
     )
-    (property "Footprint" "cap_pads:CAPPAD_7.6x7.6_Chevron_2" (id 2) (at 127 74.295 0)
+    (property "Footprint" "cap_pads:CAPPAD_7.6x7.6_Chevron_2_TopPTH" (id 2) (at 127 74.295 0)
       (effects (font (size 1.27 1.27)) hide)
     )
@@
     )
     (path "/ba1958a1-7d76-4e1e-8b73-7c7712e56926"
-      (reference "TP1") (unit 1) (value "TestPoint_Alt") (footprint "cap_pads:CAPPAD_7.6x7.6_Chevron_1")
+      (reference "TP1") (unit 1) (value "TestPoint_Alt") (footprint "cap_pads:CAPPAD_7.6x7.6_Chevron_1_TopPTH")
     )
     (path "/8b9944d7-de45-4c10-8f23-654b52f4b910"
-      (reference "TP2") (unit 1) (value "TestPoint_Alt") (footprint "cap_pads:CAPPAD_7.6x7.6_Chevron_2")
+      (reference "TP2") (unit 1) (value "TestPoint_Alt") (footprint "cap_pads:CAPPAD_7.6x7.6_Chevron_2_TopPTH")
     )
     (path "/619d42dc-7a77-4d03-bcdd-97078c405047"
-      (reference "TP3") (unit 1) (value "TestPoint_Alt") (footprint "cap_pads:CAPPAD_7.6x7.6_Chevron_2")
+      (reference "TP3") (unit 1) (value "TestPoint_Alt") (footprint "cap_pads:CAPPAD_7.6x7.6_Chevron_2_TopPTH")
     )
     (path "/b829908f-cd58-4d41-823c-96c17337397b"
-      (reference "TP4") (unit 1) (value "TestPoint_Alt") (footprint "cap_pads:CAPPAD_7.6x7.6_Chevron_2")
+      (reference "TP4") (unit 1) (value "TestPoint_Alt") (footprint "cap_pads:CAPPAD_7.6x7.6_Chevron_2_TopPTH")
     )
     (path "/625a82e9-f251-4d4b-85a0-987cbbd608cd"
-      (reference "TP5") (unit 1) (value "TestPoint_Alt") (footprint "cap_pads:CAPPAD_7.6x7.6_Chevron_2")
+      (reference "TP5") (unit 1) (value "TestPoint_Alt") (footprint "cap_pads:CAPPAD_7.6x7.6_Chevron_2_TopPTH")
     )
     (path "/bc614aae-bf8a-4524-b8fb-f2986c6a385f"
@@
     )
     (path "/b13c650d-d345-428a-ba03-fd5871ca5c98"
-      (reference "TP7") (unit 1) (value "TestPoint_Alt") (footprint "cap_pads:CAPPAD_7.6x7.6_Chevron_2_shifted")
+      (reference "TP7") (unit 1) (value "TestPoint_Alt") (footprint "cap_pads:CAPPAD_7.6x7.6_Chevron_2_TopPTH")
     )
     (path "/4e184203-7c1c-4b52-a73a-be217f4bb796"
-      (reference "TP8") (unit 1) (value "TestPoint_Alt") (footprint "cap_pads:CAPPAD_7.6x7.6_Chevron_2")
+      (reference "TP8") (unit 1) (value "TestPoint_Alt") (footprint "cap_pads:CAPPAD_7.6x7.6_Chevron_2_TopPTH")
     )
     (path "/39942e6b-3cc0-4ee7-8c07-44ca728f58d6"
-      (reference "TP9") (unit 1) (value "TestPoint_Alt") (footprint "cap_pads:CAPPAD_7.6x7.6_Chevron_2")
+      (reference "TP9") (unit 1) (value "TestPoint_Alt") (footprint "cap_pads:CAPPAD_7.6x7.6_Chevron_2_TopPTH")
     )
     (path "/f030bf22-0011-4c17-a015-6e34a85a327f"
-      (reference "TP10") (unit 1) (value "TestPoint_Alt") (footprint "cap_pads:CAPPAD_7.6x7.6_Chevron_2")
+      (reference "TP10") (unit 1) (value "TestPoint_Alt") (footprint "cap_pads:CAPPAD_7.6x7.6_Chevron_2_TopPTH")
     )
     (path "/5200f4f7-8155-455b-8d82-55039fa33a17"
-      (reference "TP11") (unit 1) (value "TestPoint_Alt") (footprint "cap_pads:CAPPAD_7.6x7.6_Chevron_2")
+      (reference "TP11") (unit 1) (value "TestPoint_Alt") (footprint "cap_pads:CAPPAD_7.6x7.6_Chevron_2_TopPTH")
     )
     (path "/1db37ab1-6540-4715-a5f1-8f515d3788c5"
-      (reference "TP12") (unit 1) (value "TestPoint_Alt") (footprint "cap_pads:CAPPAD_7.6x7.6_Chevron_3")
+      (reference "TP12") (unit 1) (value "TestPoint_Alt") (footprint "cap_pads:CAPPAD_7.6x7.6_Chevron_3_TopPTH")
     )
     (path "/c8c3ab22-4b33-4bf7-93a7-fa49e1af3364"

Commit message: updated sch and pcb with taller pads
Parts:
- TP1: footprint cap_pads:CAPPAD_7.6x7.6_Chevron_1_TopPTH -> cap_pads:CAPPADS_7.6x11.6_Chevron_1
- TP10, TP11, TP2, TP3, TP4, TP5, TP7, TP8, TP9: footprint cap_pads:CAPPAD_7.6x7.6_Chevron_2_TopPTH -> cap_pads:CAPPADS_7.6x11.6_Chevron_2
- TP12: footprint cap_pads:CAPPAD_7.6x7.6_Chevron_3_TopPTH -> cap_pads:CAPPADS_7.6x11.6_Chevron_3
- TP6: footprint cap_pads:CAPPAD_7.6x7.6_Chevron_2_shifted -> cap_pads:CAPPADS_7.6x11.6_Chevron_2
Changed lines of the file:
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@@
       (effects (font (size 1.27 1.27)) (justify left) hide)
     )
-    (property "Footprint" "cap_pads:CAPPAD_7.6x7.6_Chevron_3_TopPTH" (id 2) (at 127 79.375 0)
+    (property "Footprint" "cap_pads:CAPPADS_7.6x11.6_Chevron_3" (id 2) (at 127 79.375 0)
       (effects (font (size 1.27 1.27)) hide)
     )
@@
       (effects (font (size 1.27 1.27)) (justify left) hide)
     )
-    (property "Footprint" "cap_pads:CAPPAD_7.6x7.6_Chevron_2_TopPTH" (id 2) (at 127 71.755 0)
+    (property "Footprint" "cap_pads:CAPPADS_7.6x11.6_Chevron_2" (id 2) (at 127 71.755 0)
       (effects (font (size 1.27 1.27)) hide)
     )
@@
       (effects (font (size 1.27 1.27)) (justify left) hide)
     )
-    (property "Footprint" "cap_pads:CAPPAD_7.6x7.6_Chevron_2_TopPTH" (id 2) (at 127 69.215 0)
+    (property "Footprint" "cap_pads:CAPPADS_7.6x11.6_Chevron_2" (id 2) (at 127 69.215 0)
       (effects (font (size 1.27 1.27)) hide)
     )
@@
       (effects (font (size 1.27 1.27)) (justify left) hide)
     )
-    (property "Footprint" "cap_pads:CAPPAD_7.6x7.6_Chevron_2_TopPTH" (id 2) (at 127 76.835 0)
+    (property "Footprint" "cap_pads:CAPPADS_7.6x11.6_Chevron_2" (id 2) (at 127 76.835 0)
       (effects (font (size 1.27 1.27)) hide)
     )
@@
       (effects (font (size 1.27 1.27)) (justify left) hide)
     )
-    (property "Footprint" "cap_pads:CAPPAD_7.6x7.6_Chevron_2_TopPTH" (id 2) (at 127 56.515 0)
+    (property "Footprint" "cap_pads:CAPPADS_7.6x11.6_Chevron_2" (id 2) (at 127 56.515 0)
       (effects (font (size 1.27 1.27)) hide)
     )
@@
       (effects (font (size 1.27 1.27)) (justify left) hide)
     )
-    (property "Footprint" "cap_pads:CAPPAD_7.6x7.6_Chevron_2_TopPTH" (id 2) (at 127 61.595 0)
+    (property "Footprint" "cap_pads:CAPPADS_7.6x11.6_Chevron_2" (id 2) (at 127 61.595 0)
       (effects (font (size 1.27 1.27)) hide)
     )
@@
       (effects (font (size 1.27 1.27)) (justify left) hide)
     )
-    (property "Footprint" "cap_pads:CAPPAD_7.6x7.6_Chevron_2_TopPTH" (id 2) (at 127 53.975 0)
+    (property "Footprint" "cap_pads:CAPPADS_7.6x11.6_Chevron_2" (id 2) (at 127 53.975 0)
       (effects (font (size 1.27 1.27)) hide)
     )
@@
       (effects (font (size 1.27 1.27)) (justify left) hide)
     )
-    (property "Footprint" "cap_pads:CAPPAD_7.6x7.6_Chevron_2_TopPTH" (id 2) (at 127 66.675 0)
+    (property "Footprint" "cap_pads:CAPPADS_7.6x11.6_Chevron_2" (id 2) (at 127 66.675 0)
       (effects (font (size 1.27 1.27)) hide)
     )
@@
       (effects (font (size 1.27 1.27)) (justify left) hide)
     )
-    (property "Footprint" "cap_pads:CAPPAD_7.6x7.6_Chevron_2_TopPTH" (id 2) (at 127 59.055 0)
+    (property "Footprint" "cap_pads:CAPPADS_7.6x11.6_Chevron_2" (id 2) (at 127 59.055 0)
       (effects (font (size 1.27 1.27)) hide)
     )
@@
       (effects (font (size 1.27 1.27)) (justify left) hide)
     )
-    (property "Footprint" "cap_pads:CAPPAD_7.6x7.6_Chevron_1_TopPTH" (id 2) (at 127 51.435 0)
+    (property "Footprint" "cap_pads:CAPPADS_7.6x11.6_Chevron_1" (id 2) (at 127 51.435 0)
       (effects (font (size 1.27 1.27)) hide)
     )
@@
       (effects (font (size 1.27 1.27)) (justify left) hide)
     )
-    (property "Footprint" "cap_pads:CAPPAD_7.6x7.6_Chevron_2_shifted" (id 2) (at 127 64.135 0)
+    (property "Footprint" "cap_pads:CAPPADS_7.6x11.6_Chevron_2" (id 2) (at 127 64.135 0)
       (effects (font (size 1.27 1.27)) hide)
     )
@@
       (effects (font (size 1.27 1.27)) (justify left) hide)
     )
-    (property "Footprint" "cap_pads:CAPPAD_7.6x7.6_Chevron_2_TopPTH" (id 2) (at 127 74.295 0)
+    (property "Footprint" "cap_pads:CAPPADS_7.6x11.6_Chevron_2" (id 2) (at 127 74.295 0)
       (effects (font (size 1.27 1.27)) hide)
     )
@@
     )
     (path "/ba1958a1-7d76-4e1e-8b73-7c7712e56926"
-      (reference "TP1") (unit 1) (value "TestPoint_Alt") (footprint "cap_pads:CAPPAD_7.6x7.6_Chevron_1_TopPTH")
+      (reference "TP1") (unit 1) (value "TestPoint_Alt") (footprint "cap_pads:CAPPADS_7.6x11.6_Chevron_1")
     )
     (path "/8b9944d7-de45-4c10-8f23-654b52f4b910"
-      (reference "TP2") (unit 1) (value "TestPoint_Alt") (footprint "cap_pads:CAPPAD_7.6x7.6_Chevron_2_TopPTH")
+      (reference "TP2") (unit 1) (value "TestPoint_Alt") (footprint "cap_pads:CAPPADS_7.6x11.6_Chevron_2")
     )
     (path "/619d42dc-7a77-4d03-bcdd-97078c405047"
-      (reference "TP3") (unit 1) (value "TestPoint_Alt") (footprint "cap_pads:CAPPAD_7.6x7.6_Chevron_2_TopPTH")
+      (reference "TP3") (unit 1) (value "TestPoint_Alt") (footprint "cap_pads:CAPPADS_7.6x11.6_Chevron_2")
     )
     (path "/b829908f-cd58-4d41-823c-96c17337397b"
-      (reference "TP4") (unit 1) (value "TestPoint_Alt") (footprint "cap_pads:CAPPAD_7.6x7.6_Chevron_2_TopPTH")
+      (reference "TP4") (unit 1) (value "TestPoint_Alt") (footprint "cap_pads:CAPPADS_7.6x11.6_Chevron_2")
     )
     (path "/625a82e9-f251-4d4b-85a0-987cbbd608cd"
-      (reference "TP5") (unit 1) (value "TestPoint_Alt") (footprint "cap_pads:CAPPAD_7.6x7.6_Chevron_2_TopPTH")
+      (reference "TP5") (unit 1) (value "TestPoint_Alt") (footprint "cap_pads:CAPPADS_7.6x11.6_Chevron_2")
     )
     (path "/bc614aae-bf8a-4524-b8fb-f2986c6a385f"
-      (reference "TP6") (unit 1) (value "TestPoint_Alt") (footprint "cap_pads:CAPPAD_7.6x7.6_Chevron_2_shifted")
+      (reference "TP6") (unit 1) (value "TestPoint_Alt") (footprint "cap_pads:CAPPADS_7.6x11.6_Chevron_2")
     )
     (path "/b13c650d-d345-428a-ba03-fd5871ca5c98"
-      (reference "TP7") (unit 1) (value "TestPoint_Alt") (footprint "cap_pads:CAPPAD_7.6x7.6_Chevron_2_TopPTH")
+      (reference "TP7") (unit 1) (value "TestPoint_Alt") (footprint "cap_pads:CAPPADS_7.6x11.6_Chevron_2")
     )
     (path "/4e184203-7c1c-4b52-a73a-be217f4bb796"
-      (reference "TP8") (unit 1) (value "TestPoint_Alt") (footprint "cap_pads:CAPPAD_7.6x7.6_Chevron_2_TopPTH")
+      (reference "TP8") (unit 1) (value "TestPoint_Alt") (footprint "cap_pads:CAPPADS_7.6x11.6_Chevron_2")
     )
     (path "/39942e6b-3cc0-4ee7-8c07-44ca728f58d6"
-      (reference "TP9") (unit 1) (value "TestPoint_Alt") (footprint "cap_pads:CAPPAD_7.6x7.6_Chevron_2_TopPTH")
+      (reference "TP9") (unit 1) (value "TestPoint_Alt") (footprint "cap_pads:CAPPADS_7.6x11.6_Chevron_2")
     )
     (path "/f030bf22-0011-4c17-a015-6e34a85a327f"
-      (reference "TP10") (unit 1) (value "TestPoint_Alt") (footprint "cap_pads:CAPPAD_7.6x7.6_Chevron_2_TopPTH")
+      (reference "TP10") (unit 1) (value "TestPoint_Alt") (footprint "cap_pads:CAPPADS_7.6x11.6_Chevron_2")
     )
     (path "/5200f4f7-8155-455b-8d82-55039fa33a17"
-      (reference "TP11") (unit 1) (value "TestPoint_Alt") (footprint "cap_pads:CAPPAD_7.6x7.6_Chevron_2_TopPTH")
+      (reference "TP11") (unit 1) (value "TestPoint_Alt") (footprint "cap_pads:CAPPADS_7.6x11.6_Chevron_2")
     )
     (path "/1db37ab1-6540-4715-a5f1-8f515d3788c5"
-      (reference "TP12") (unit 1) (value "TestPoint_Alt") (footprint "cap_pads:CAPPAD_7.6x7.6_Chevron_3_TopPTH")
+      (reference "TP12") (unit 1) (value "TestPoint_Alt") (footprint "cap_pads:CAPPADS_7.6x11.6_Chevron_3")
     )
     (path "/c8c3ab22-4b33-4bf7-93a7-fa49e1af3364"

Commit message: 4pin, IRQ LED
Parts:
- added D1: RED, LED_SMD:LED_0805_2012Metric, symbol Device:LED_Small
- added R4: 10kΩ, Resistor_SMD:R_0805_2012Metric, symbol Device:R_Small
- J1: footprint Connector_JST:JST_SUR_SM05B-SURS-TF_1x05-1MP_P0.80mm_Horizontal -> Connector_JST:JST_SUR_SM04B-SURS-TF_1x04-1MP_P0.80mm_Horizontal; symbol Connector_Generic:Conn_01x05 -> Connector_Generic:Conn_01x04
Connections:
- net +3V3: now also R4.1
- net GND: now also J1.4 (Pin_4); no longer J1.5 (Pin_5)
- net INT: no longer names the net of U1.1 (~{IRQ})
- net INT: now also D1.1 (K); no longer J1.4 (Pin_4)
- new net: D1.2 (A), R4.2
Other:
- moved on the sheet: JP1, JP2, JP3, JP4, R1
